File: elec/layouts/default/default.kicad_pcb (KiCad board)
At the start: 2 copper layers, 20 parts, among them U1 1µF ±10% 25V X5R, U10 330kΩ ±1% 62.5mW, U11 1kΩ ±1% 62.5mW, U12 10kΩ ±1% 62.5mW, U13 1kΩ ±1% 62.5mW, U14 1kΩ ±1% 62.5mW, U15 10mΩ ±1% 1W, U2 10µF ±20% 6.3V X5R, U3 100nF ±10% 16V X7R, U4 4.7µF ±10% 10V X5R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

Commit message: changed layouts to original layout folder name, fixed layout syncing
Connections:
- net A renamed G
- net cathode renamed VOUT
- D1 pad 1: C -> D
- U11 pad 1: C -> S
- U16 pad 1: C -> S
- U2 pad 1: C -> S
- U8 pad 2: C -> S
Changed lines of the file:
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@@
     )
     (net 0 "")
-    (net 1 "C")
+    (net 1 "S")
     (net 2 "VCTRL")
     (net 3 "ICTRL_PLUS")
-    (net 4 "A")
+    (net 4 "G")
     (net 5 "ICTRL_MINUS")
     (net 6 "hv")
     (net 7 "gnd")
-    (net 8 "cathode")
+    (net 8 "VOUT")
     (net 9 "LX")
-    (net 10 "D")
     (net 11 "XSHUT")
+    (net 12 "D")
     (footprint "lib:SOT-23-6_L2.9-W1.6-P0.95-LS2.8-BR"
         (layer "F.Cu")
@@
             (drill 0.9000235999999999)
             (layers "*.Cu" "*.Mask")
-            (net 10 "D")
+            (net 12 "D")
         )
     )
@@
             (size 0.8 0.9)
             (layers "F.Cu" "F.Paste" "F.Mask")
-            (net 1 "C")
+            (net 1 "S")
         )
     )
@@
             (size 0.57 0.54)
             (layers "F.Cu" "F.Paste" "F.Mask")
-            (net 4 "A")
+            (net 4 "G")
         )
     )
@@
             (size 0.57 0.54)
             (layers "F.Cu" "F.Paste" "F.Mask")
-            (net 8 "cathode")
+            (net 8 "VOUT")
         )
         (pad "1" smd rect
@@
             (size 1 0.8)
             (layers "F.Cu" "F.Paste" "F.Mask")
-            (net 1 "C")
+            (net 1 "S")
         )
         (pad "3" smd rect
@@
             (size 1 0.8)
             (layers "F.Cu" "F.Paste" "F.Mask")
-            (net 10 "D")
+            (net 12 "D")
         )
         (pad "1" smd rect
@@
             (size 1 0.8)
             (layers "F.Cu" "F.Paste" "F.Mask")
-            (net 4 "A")
+            (net 4 "G")
         )
     )
@@
             (size 0.35 1.45)
             (layers "F.Cu" "F.Paste" "F.Mask")
-            (net 8 "cathode")
+            (net 8 "VOUT")
         )
         (pad "8" smd oval
@@
             (size 0.8 0.9)
             (layers "F.Cu" "F.Paste" "F.Mask")
-            (net 8 "cathode")
+            (net 8 "VOUT")
         )
     )
@@
             (size 0.8 0.8)
             (layers "F.Cu" "F.Paste" "F.Mask")
-            (net 1 "C")
+            (net 12 "D")
         )
         (pad "2" smd rect
@@
             (size 0.8 0.8)
             (layers "F.Cu" "F.Paste" "F.Mask")
-            (net 4 "A")
+            (net 4 "G")
         )
     )
@@
             (size 0.57 0.54)
             (layers "F.Cu" "F.Paste" "F.Mask")
-            (net 1 "C")
+            (net 1 "S")
         )
     )
@@
             (size 1.21 1.7)
             (layers "F.Cu" "F.Paste" "F.Mask")
-            (net 8 "cathode")
+            (net 8 "VOUT")
         )
     )
@@
             (size 1.55 5.6)
             (layers "F.Cu" "F.Paste" "F.Mask")
-            (net 1 "C")
+            (net 1 "S")
         )
     )
