File: elec/layout/default/default.kicad_pcb (KiCad board)
At the start: 2 copper layers, 23.9 x 13.7 mm, 23 parts, among them U2 100nF ±10% 16V X7R, U5 10µF ±20% 6.3V X5R, U6 10kΩ ±1% 62.5mW

Commit message: updated files, layout looked unaltered
Connections:
- net A renamed anode
- net Vpvr-VCC renamed Vpv
- net XSHUT renamed MPP_SET
- net power_shim-VCC renamed Vbat
Routing:
- net (no net): track 0.00 -> 30.1 mm, vias 0 -> 2
- net Vbat: track 22.9 -> 0.00 mm, vias 2 -> 0
- net _1: track 7.19 -> 0.00 mm
Changed lines of the file:
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@@
     (net 0 "")
     (net 1 "ICTRL_MINUS")
-    (net 2 "XSHUT")
+    (net 2 "MPP_SET")
     (net 3 "ICTRL_PLUS")
     (net 4 "LX")
     (net 5 "VOUT")
     (net 6 "VCTRL")
-    (net 7 "power_shim-VCC")
-    (net 8 "Vpvr-VCC")
+    (net 8 "Vpv")
     (net 9 "VDD")
     (net 10 "power_shim-GND")
     (net 11 "Vbatr-GND")
-    (net 12 "A")
-    (net 13 "_1")
+    (net 12 "anode")
+    (net 15 "Vbat")
+    (net 16 "_1")
     (footprint "TECH_PUBLIC_SRV05_4_P_T7:SOT-23-6_L2.9-W1.6-P0.95-LS2.8-BR"
         (layer "F.Cu")
@@
             (size 0.57 0.54)
             (layers "F.Cu" "F.Paste" "F.Mask")
-            (net 7 "power_shim-VCC")
+            (net 15 "Vbat")
         )
         (model "${KIPRJMOD}/../../src/parts/UNI_ROYAL_0402WGF1004TCE/R0402_L1.0-W0.5-H0.4.step"
@@
             (drill 0.9000235999999999)
             (layers "*.Cu" "*.Mask")
-            (net 8 "Vpvr-VCC")
+            (net 8 "Vpv")
         )
         (model "${KIPRJMOD}/../../src/parts/JST_Sales_America_B2B_PH_K_S_LF__SN/CONN-TH_PH2.00-LI-2P.step"
@@
             (size 0.81 0.86)
             (layers "F.Cu" "F.Paste" "F.Mask")
-            (net 13 "_1")
+            (net 16 "_1")
         )
         (pad "1" smd rect
@@
             (size 0.81 0.86)
             (layers "F.Cu" "F.Paste" "F.Mask")
-            (net 7 "power_shim-VCC")
+            (net 15 "Vbat")
         )
         (model "${KIPRJMOD}/../../src/parts/Littelfuse_0603L150SLYR/F0603_L1.7-W0.9-H0.7.step"
@@
             (size 0.8 0.9)
             (layers "F.Cu" "F.Paste" "F.Mask")
-            (net 8 "Vpvr-VCC")
+            (net 8 "Vpv")
         )
         (model "${KIPRJMOD}/../../src/parts/Samsung_Electro_Mechanics_CL10A106MQ8NNNC/C0603_L1.6-W0.8-H0.8.step"
@@
             (drill 0.9000235999999999)
             (layers "*.Cu" "*.Mask")
-            (net 7 "power_shim-VCC")
+            (net 15 "Vbat")
         )
         (model "${KIPRJMOD}/../../src/parts/JST_Sales_America_B2B_PH_K_S_LF__SN/CONN-TH_PH2.00-LI-2P.step"
@@
             (size 0.79 0.54)
             (layers "F.Cu" "F.Paste" "F.Mask")
-            (net 2 "XSHUT")
+            (net 2 "MPP_SET")
         )
         (model "${KIPRJMOD}/../../src/parts/Samsung_Electro_Mechanics_CL05B104KO5NNNC/C0402_L1.0-W0.5-H0.5.step"
@@
             (size 0.35 1.45)
             (layers "F.Cu" "F.Paste" "F.Mask")
-            (net 2 "XSHUT")
+            (net 2 "MPP_SET")
         )
         (pad "2" smd oval
@@
             (size 0.35 1.45)
             (layers "F.Cu" "F.Paste" "F.Mask")
-            (net 2 "XSHUT")
+            (net 2 "MPP_SET")
         )
         (pad "7" smd oval
@@
             (size 0.57 0.54)
             (layers "F.Cu" "F.Paste" "F.Mask")
-            (net 7 "power_shim-VCC")
+            (net 15 "Vbat")
         )
         (pad "1" smd rect
@@
             (size 1.55 5.6)
             (layers "F.Cu" "F.Paste" "F.Mask")
-            (net 8 "Vpvr-VCC")
+            (net 8 "Vpv")
         )
         (model "${KIPRJMOD}/../../src/parts/Coilcraft_XAL6060_103MEC/IND-SMD_L6.6-W6.4-H2.9.step"
@@
             (size 1.1 1)
             (layers "F.Cu" "F.Paste" "F.Mask")
-            (net 12 "A")
+            (net 12 "anode")
         )
         (model "${KIPRJMOD}/../../src/parts/GOODWORK_B5819W/SOD-123F_L2.7-W1.6-LS3.8-RD-1.STEP"
@@
             (size 1.21 1.7)
             (layers "F.Cu" "F.Paste" "F.Mask")
-            (net 7 "power_shim-VCC")
+            (net 15 "Vbat")
         )
         (pad "1" smd rect
@@
             (drill 0.9000235999999999)
             (layers "*.Cu" "*.Mask")
-            (net 12 "A")
+            (net 12 "anode")
         )
         (pad "1" thru_hole circle
@@
             (drill 0.9000235999999999)
             (layers "*.Cu" "*.Mask")
-            (net 13 "_1")
+            (net 16 "_1")
         )
         (model "${KIPRJMOD}/../../src/parts/JST_Sales_America_B2B_PH_K_S_LF__SN/CONN-TH_PH2.00-LI-2P.step"
@@
             (size 0.57 0.54)
             (layers "F.Cu" "F.Paste" "F.Mask")
-            (net 7 "power_shim-VCC")
+            (net 15 "Vbat")
         )
         (pad "1" smd rect
@@
             (size 0.8 0.9)
             (layers "F.Cu" "F.Paste" "F.Mask")
-            (net 7 "power_shim-VCC")
+            (net 15 "Vbat")
         )
         (model "${KIPRJMOD}/../../src/parts/Samsung_Electro_Mechanics_CL10A106MQ8NNNC/C0603_L1.6-W0.8-H0.8.step"
@@
             (size 0.57 0.54)
             (layers "F.Cu" "F.Paste" "F.Mask")
-            (net 2 "XSHUT")
+            (net 2 "MPP_SET")
         )
         (pad "1" smd rect
@@
             (size 0.57 0.54)
             (layers "F.Cu" "F.Paste" "F.Mask")
-            (net 8 "Vpvr-VCC")
+            (net 8 "Vpv")
         )
         (model "${KIPRJMOD}/../../src/parts/UNI_ROYAL_0402WGF1001TCE/R0402_L1.0-W0.5-H0.4.step"
@@
         (drill 0.4)
         (layers "F.Cu" "B.Cu")
-        (net 7)
+        (net 0)
     )
     (via
@@
         (drill 0.4)
         (layers "F.Cu" "B.Cu")
-        (net 7)
+        (net 0)
     )
     (via
@@
         (end 85.5 50.8575)
         (width 0.635)
-        (net 7)
+        (net 0)
         (layer "F.Cu")
     )
@@
         (end 86.91125 51.67875)
         (width 0.635)
-        (net 7)
+        (net 0)
         (layer "F.Cu")
     )
@@
         (end 85.9925 53.4575)
         (width 0.635)
-        (net 7)
+        (net 0)
         (layer "F.Cu")
     )
@@
         (end 84.6 52.15)
         (width 0.25)
-        (net 7)
+        (net 0)
         (layer "F.Cu")
     )
@@
         (end 87.6425 53.5)
         (width 0.5)
-        (net 7)
+        (net 0)
         (layer "F.Cu")
     )
@@
         (end 84.5 52.25)
         (width 0.25)
-        (net 7)
+        (net 0)
         (layer "F.Cu")
     )
@@
         (end 85.0425 50.2)
         (width 0.635)
-        (net 7)
+        (net 0)
         (layer "F.Cu")
     )
@@
         (end 88.1 53.4575)
         (width 0.635)
-        (net 7)
+        (net 0)
         (layer "F.Cu")
     )
@@
         (end 83.9425 49.1)
         (width 0.635)
-        (net 7)
+        (net 0)
         (layer "F.Cu")
     )
@@
         (end 85.9 53.55)
         (width 0.635)
-        (net 7)
+        (net 0)
         (layer "F.Cu")
     )
@@
         (end 86.32125 51.67875)
         (width 0.635)
-        (net 7)
+        (net 0)
         (layer "F.Cu")
     )
@@
         (end 85.8 51.2)
         (width 0.635)
-        (net 7)
+        (net 0)
         (layer "F.Cu")
     )
@@
         (end 85.5 50.9)
         (width 0.635)
-        (net 7)
+        (net 0)
         (layer "F.Cu")
     )
@@
         (end 85.8 51.65)
         (width 0.25)
-        (net 7)
+        (net 0)
         (layer "F.Cu")
     )
@@
         (end 85.5 50.2)
         (width 0.635)
-        (net 7)
+        (net 0)
         (layer "F.Cu")
     )
@@
         (end 86.32125 53.4575)
         (width 0.635)
-        (net 7)
+        (net 0)
         (layer "F.Cu")
     )
@@
         (end 90.0425 46.6)
         (width 0.25)
-        (net 7)
+        (net 0)
         (layer "F.Cu")
     )
@@
         (end 89.9825 46.54)
         (width 0.25)
-        (net 7)
+        (net 0)
         (layer "F.Cu")
     )
@@
         (end 84.4 53.55)
         (width 0.635)
-        (net 7)
+        (net 0)
         (layer "F.Cu")
     )
@@
         (end 86.94 51.65)
         (width 0.635)
-        (net 7)
+        (net 0)
         (layer "F.Cu")
     )
@@
         (end 85.3 52.15)
         (width 0.25)
-        (net 7)
+        (net 0)
         (layer "F.Cu")
     )
@@
         (end 91 46.6)
         (width 0.25)
-        (net 7)
+        (net 0)
         (layer "B.Cu")
     )
@@
         (end 85.575 50.6)
         (width 0.25)
-        (net 7)
+        (net 0)
         (layer "B.Cu")
     )
@@
         (end 91 47.4)
         (width 0.25)
-        (net 7)
+        (net 0)
         (layer "B.Cu")
     )
@@
         (end 85.5 50.525)
         (width 0.25)
-        (net 7)
+        (net 0)
         (layer "B.Cu")
     )
@@
         (end 87.8 50.6)
         (width 0.25)
-        (net 7)
+        (net 0)
         (layer "B.Cu")
     )
@@
         (end 78 52.7)
         (width 0.5)
-        (net 13)
+        (net 0)
         (layer "F.Cu")
     )
@@
         (end 80.3 52.988162)
         (width 0.5)
-        (net 13)
+        (net 0)
         (layer "F.Cu")
     )
@@
         (end 82.9 53.55)
         (width 0.5)
-        (net 13)
+        (net 0)
         (layer "F.Cu")
     )
@@
         (end 80.011838 52.7)
         (width 0.5)
-        (net 13)
+        (net 0)
         (layer "F.Cu")
     )
@@
         (end 77.3 53.9)
         (width 0.5)
-        (net 13)
+        (net 0)
         (layer "F.Cu")
     )
@@
         (end 76.9 54)
         (width 0.25)
-        (net 13)
+        (net 0)
         (layer "F.Cu")
     )
@@
         (end 77.2 54)
         (width 0.5)
-        (net 13)
+        (net 0)
         (layer "F.Cu")
     )
@@
         (end 80.85 53.55)
         (width 0.5)
-        (net 13)
+        (net 0)
         (layer "F.Cu")
     )
@@
         (end 77.3 53.4)
         (width 0.5)
-        (net 13)
+        (net 0)
         (layer "F.Cu")
     )

Commit message: update! works with current ato version
Parts:
- moved R2 0.20 mm to (73.8, 51.3)
Routing:
- net (no net): track 30.1 -> 0.00 mm, vias 2 -> 0
- net Vbat: track 0.00 -> 22.9 mm, vias 0 -> 2
- net _1: track 0.00 -> 7.19 mm
- net power_shim-GND: vias 12 -> 11
Other:
- board text added: "ICTRL"
- board text added: "LION"
- board text added: "SPV1040"
